File: CANFD/4CAN.kicad_pcb (KiCad board)
At the start: 2 copper layers, 44 parts, among them J1 , J2 , J3 , J4 , J5 , SW1 , U1 , U2 , U3 , U4 , U5 , U6 , U7 , U8 , U9 

Commit message: latest version of 4CAN-FD design files
Parts:
- D2, D3, D4: value (none) -> .
- U4, U5, U6, U7, U8, U9: value (none) -> (none)
Connections:
-   pad 8: (no net) -> Net-(J1-Pad7)
- C1 pad 1: (no net) -> VCC
- C1 pad 2: (no net) -> GND
- C10 pad 1: (no net) -> VCC
- C10 pad 2: (no net) -> GND
- C11 pad 1: (no net) -> VCC
- C11 pad 2: (no net) -> GND
- C12 pad 1: (no net) -> VCC
- C12 pad 2: (no net) -> GND
- C13 pad 1: (no net) -> VCC
- C13 pad 2: (no net) -> GND
- C2 pad 1: (no net) -> VCC
- C2 pad 2: (no net) -> GND
- C3 pad 1: (no net) -> GND
- C3 pad 2: (no net) -> VCC
- C5 pad 1: (no net) -> VCC
- C5 pad 2: (no net) -> GND
- C6 pad 1: (no net) -> VCC
- C6 pad 2: (no net) -> GND
- C7 pad 1: (no net) -> VCC
- C7 pad 2: (no net) -> GND
- C8 pad 1: (no net) -> VCC
- C8 pad 2: (no net) -> GND
- C9 pad 1: (no net) -> VCC
- C9 pad 2: (no net) -> GND
- D3 pad 1: (no net) -> GND
- D4 pad 1: (no net) -> GND
- D5 pad 1: (no net) -> Net-(D5-Pad~)
- D5 pad 2: (no net) -> Net-(D5-Pad~)
- D5 pad 3: (no net) -> GND
- D6 pad 1: (no net) -> Net-(D6-Pad~)
- D6 pad 2: (no net) -> Net-(D6-Pad~)
- D6 pad 3: (no net) -> GND
- D7 pad 1: (no net) -> Net-(D7-Pad~)
- D7 pad 2: (no net) -> Net-(D7-Pad~)
- D7 pad 3: (no net) -> GND
- D8 pad 1: (no net) -> Net-(D8-Pad~)
- D8 pad 2: (no net) -> Net-(D8-Pad~)
- D8 pad 3: (no net) -> GND
- J1 pad 1: (no net) -> VCC
- J1 pad 10: (no net) -> RX
- J1 pad 11: (no net) -> Net-(J1-Pad11)
- J1 pad 12: (no net) -> GND
- J1 pad 13: (no net) -> /SPI1-CE1
- J1 pad 14: (no net) -> GND
- J1 pad 15: (no net) -> GND
- J1 pad 16: (no net) -> GND
- J1 pad 17: (no net) -> VCC
- J1 pad 19: (no net) -> /SPI-MOSI
- J1 pad 2: (no net) -> VCC
- J1 pad 20: (no net) -> GND
- J1 pad 21: (no net) -> /SPI-MISO
- J1 pad 22: (no net) -> GND
- J1 pad 23: (no net) -> /SPI-SCLK
- J1 pad 24: (no net) -> GND
- J1 pad 25: (no net) -> GND
- J1 pad 26: (no net) -> GND
- J1 pad 27: (no net) -> Net-(J1-Pad27)
- J1 pad 28: (no net) -> Net-(J1-Pad28)
- J1 pad 29: (no net) -> Net-(J1-Pad29)
- J1 pad 3: (no net) -> VCC
- J1 pad 30: (no net) -> GND
- J1 pad 31: (no net) -> Net-(D3-Pad~)
- J1 pad 32: (no net) -> Net-(J1-Pad32)
- J1 pad 33: (no net) -> Net-(J1-Pad33)
- J1 pad 34: (no net) -> GND
- J1 pad 35: (no net) -> /SPI-MISO
- J1 pad 36: (no net) -> Net-(J1-Pad36)
- J1 pad 37: (no net) -> Net-(D4-Pad~)
- J1 pad 38: (no net) -> GND
- J1 pad 39: (no net) -> GND
- J1 pad 4: (no net) -> VCC
- J1 pad 5: (no net) -> Net-(J1-Pad5)
- J1 pad 6: (no net) -> GND
- J1 pad 7: (no net) -> Net-(J1-Pad7)
- J1 pad 8: (no net) -> TX
- J1 pad 9: (no net) -> GND
- J1 pad None: (no net) -> /SPI-MISO
- J2 pad 1: (no net) -> Net-(D5-Pad~)
- J2 pad 2: (no net) -> Net-(D5-Pad~)
- J2 pad 3: (no net) -> GND
- J3 pad 1: (no net) -> Net-(D6-Pad~)
- J3 pad 2: (no net) -> Net-(D6-Pad~)
- J3 pad 3: (no net) -> GND
- J4 pad 1: (no net) -> Net-(D7-Pad~)
- J4 pad 2: (no net) -> Net-(D7-Pad~)
- J4 pad 3: (no net) -> GND
- J5 pad 1: (no net) -> Net-(D8-Pad~)
- J5 pad 2: (no net) -> Net-(D8-Pad~)
- J5 pad 3: (no net) -> GND
- R1 pad 1: (no net) -> VCC
- R1 pad 2: (no net) -> GND
- R2 pad 1: (no net) -> VCC
- R2 pad 2: (no net) -> GND
- R3 pad 1: (no net) -> VCC
- R3 pad 2: (no net) -> GND
- R4 pad 1: (no net) -> VCC
- R4 pad 2: (no net) -> Net-(J1-Pad11)
- R5 pad 1: (no net) -> Net-(D5-Pad~)
- R5 pad 2: (no net) -> Net-(R5-Pad1)
- R6 pad 1: (no net) -> Net-(D6-Pad~)
- R6 pad 2: (no net) -> Net-(R6-Pad1)
- R7 pad 1: (no net) -> Net-(D7-Pad~)
- R7 pad 2: (no net) -> Net-(R7-Pad1)
- R8 pad 1: (no net) -> Net-(D8-Pad~)
- R8 pad 2: (no net) -> Net-(R8-Pad1)
- SW1 pad 1: (no net) -> Net-(R5-Pad1)
- SW1 pad 2: (no net) -> Net-(R6-Pad1)
- SW1 pad 3: (no net) -> Net-(R7-Pad1)
- SW1 pad 4: (no net) -> Net-(R8-Pad1)
- SW1 pad 5: (no net) -> Net-(D8-Pad~)
- SW1 pad 6: (no net) -> Net-(D7-Pad~)
- SW1 pad 7: (no net) -> Net-(D6-Pad~)
- SW1 pad 8: (no net) -> Net-(D5-Pad~)
- U1 pad 1: (no net) -> VCC
- U1 pad 2: (no net) -> GND
- U1 pad 3: (no net) -> Net-(U1-Pad3)
- U1 pad 4: (no net) -> VCC
- U2 pad 1: (no net) -> Net-(U2-Pad1)
- U2 pad 10: (no net) -> /SPI-SCLK
- U2 pad 11: (no net) -> /SPI-MOSI
- U2 pad 12: (no net) -> /SPI-MISO
- U2 pad 13: (no net) -> GND
- U2 pad 14: (no net) -> VCC
- U2 pad 2: (no net) -> Net-(U2-Pad2)
- U2 pad 5: (no net) -> Net-(U2-Pad5)
- U2 pad 6: (no net) -> Net-(U1-Pad3)
- U2 pad 7: (no net) -> GND
- U2 pad 8: (no net) -> Net-(U2-Pad8)
- U2 pad 9: (no net) -> Net-(U2-Pad9)
- U3 pad 1: (no net) -> Net-(U3-Pad1)
- U3 pad 10: (no net) -> /SPI-SCLK
- U3 pad 11: (no net) -> /SPI-MOSI
- U3 pad 12: (no net) -> /SPI-MISO
- U3 pad 13: (no net) -> GND
- U3 pad 14: (no net) -> VCC
- U3 pad 2: (no net) -> Net-(U3-Pad2)
- U3 pad 3: (no net) -> Net-(U3-Pad3)
- U3 pad 5: (no net) -> Net-(U3-Pad5)
- U3 pad 6: (no net) -> Net-(U1-Pad3)
- U3 pad 7: (no net) -> GND
- U3 pad 8: (no net) -> Net-(U3-Pad8)
- U3 pad 9: (no net) -> Net-(U3-Pad9)
- U4 pad 1: (no net) -> Net-(U4-Pad1)
- U4 pad 10: (no net) -> /SPI-SCLK
- U4 pad 11: (no net) -> GND
- U4 pad 12: (no net) -> /SPI-MISO
- U4 pad 13: (no net) -> GND
- U4 pad 14: (no net) -> VCC
- U4 pad 2: (no net) -> Net-(U4-Pad2)
- U4 pad 3: (no net) -> Net-(U4-Pad3)
- U4 pad 5: (no net) -> Net-(U4-Pad5)
- U4 pad 6: (no net) -> Net-(U1-Pad3)
- U4 pad 7: (no net) -> GND
- U4 pad 8: (no net) -> Net-(U4-Pad8)
- U4 pad 9: (no net) -> Net-(U4-Pad9)
- U5 pad 1: (no net) -> Net-(U5-Pad1)
- U5 pad 10: (no net) -> /SPI-SCLK
- U5 pad 11: (no net) -> GND
- U5 pad 12: (no net) -> /SPI-MISO
- U5 pad 13: (no net) -> Net-(J1-Pad11)
- U5 pad 14: (no net) -> VCC
- U5 pad 2: (no net) -> Net-(U5-Pad2)
- U5 pad 3: (no net) -> Net-(U5-Pad3)
- U5 pad 5: (no net) -> Net-(U5-Pad5)
- U5 pad 6: (no net) -> Net-(U1-Pad3)
- U5 pad 7: (no net) -> GND
- U5 pad 8: (no net) -> Net-(U5-Pad8)
- U5 pad 9: (no net) -> Net-(U5-Pad9)
- U6 pad 1: (no net) -> Net-(U2-Pad1)
- U6 pad 2: (no net) -> GND
- U6 pad 3: (no net) -> VCC
- U6 pad 4: (no net) -> Net-(U2-Pad2)
- U6 pad 6: (no net) -> Net-(D5-Pad~)
- U6 pad 7: (no net) -> Net-(D5-Pad~)
- U6 pad 8: (no net) -> GND
- U7 pad 1: (no net) -> Net-(U3-Pad1)
- U7 pad 2: (no net) -> GND
- U7 pad 3: (no net) -> VCC
- U7 pad 4: (no net) -> Net-(U3-Pad2)
- U7 pad 6: (no net) -> Net-(D6-Pad~)
- U7 pad 7: (no net) -> Net-(D6-Pad~)
- U7 pad 8: (no net) -> GND
- U8 pad 1: (no net) -> Net-(U4-Pad1)
- U8 pad 2: (no net) -> GND
- U8 pad 3: (no net) -> VCC
- U8 pad 4: (no net) -> Net-(U4-Pad2)
- U8 pad 6: (no net) -> Net-(D7-Pad~)
- U8 pad 7: (no net) -> Net-(D7-Pad~)
- U8 pad 8: (no net) -> GND
- U9 pad 1: (no net) -> Net-(U5-Pad1)
- U9 pad 2: (no net) -> GND
- U9 pad 3: (no net) -> VCC
- U9 pad 4: (no net) -> Net-(U5-Pad2)
- U9 pad 6: (no net) -> Net-(D8-Pad~)
- U9 pad 7: (no net) -> Net-(D8-Pad~)
- U9 pad 8: (no net) -> GND
Routing:
- net (no net): track 1951.0 -> 180.0 mm, vias 91 -> 13
- net GND: track 0.00 -> 491.1 mm, vias 0 -> 32
- net VCC: track 0.00 -> 299.3 mm, vias 0 -> 16
- net Net-(D5-Pad~): track 0.00 -> 109.8 mm, vias 0 -> 1
- net Net-(D6-Pad~): track 0.00 -> 97.7 mm, vias 0 -> 3
- net Net-(D7-Pad~): track 0.00 -> 84.5 mm, vias 0 -> 3
- net /SPI-MISO: track 0.00 -> 70.7 mm, vias 0 -> 6
- net /SPI-SCLK: track 0.00 -> 69.4 mm, vias 0 -> 5
- net Net-(J1-Pad7): track 0.00 -> 67.6 mm, vias 0 -> 2
- net Net-(D8-Pad~): track 0.00 -> 67.5 mm, vias 0 -> 3
- net Net-(U1-Pad3): track 0.00 -> 66.3 mm, vias 0 -> 5
- net Net-(R5-Pad1): track 0.00 -> 52.1 mm
- net /SPI1-CE1: track 0.00 -> 44.7 mm
- net Net-(R6-Pad1): track 0.00 -> 35.9 mm
- net /SPI-MOSI: track 0.00 -> 31.9 mm, vias 0 -> 2
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Other:
- rule trace_min: 0.2 -> 0
