File: CANFD/4CAN.sch (KiCad schematic (older format))
At the start: 44 parts, among them J1 NPTC202KFMS-RC, J2 ED555_2DS, J3 ED555_2DS, J4 ED555_2DS, J5 ED555_2DS, SW1 218-4LPSTR, U1 , U2 MCP2518FDT-H_SL, U3 MCP2518FDT-H_SL, U4 MCP2518FDT-H_SL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

Commit message: latest version of 4CAN-FD design files
Parts:
- C1: symbol 4CAN-rescue:F930J227MNC-2020-06-11_20-40-41 -> 4CAN-rescue:F930J227MNC-2020-06-11_20-40-41-4CAN-rescue
- C10, C11, C12, C13, C2, C3, C5, C6, C7, C8, C9: symbol 4CAN-rescue:C0805Y103K1RACAUTO-2020-06-11_20-43-35 -> 4CAN-rescue:C0805Y103K1RACAUTO-2020-06-11_20-43-35-4CAN-rescue
- D1, D2, D3, D4: symbol 4CAN-rescue:.-XZMDKVG55W-8 -> 4CAN-rescue:.-XZMDKVG55W-8-4CAN-rescue
- J2, J3, J4, J5: symbol 4CAN-rescue:ED555_2DS-2020-06-09_21-20-13 -> 4CAN-rescue:ED555_2DS-2020-06-09_21-20-13-4CAN-rescue
- R1, R2, R3, R4, R5, R6, R7, R8: symbol 4CAN-rescue:RC0805FR-07120RL-2020-06-09_18-29-32 -> 4CAN-rescue:RC0805FR-07120RL-2020-06-09_18-29-32-4CAN-rescue
Connections:
- new net: D1.~ (C), RP503.~
Changed lines of the file:
@@
 	8900 11300 5950 11300
 $Comp
-L 4CAN-rescue:.-XZMDKVG55W-8 D1
+L 4CAN-rescue:.-XZMDKVG55W-8-4CAN-rescue D1
 U 1 1 5F034D42
 P 6750 7100
@@
 $EndComp
 $Comp
-L 4CAN-rescue:.-XZMDKVG55W-8 D2
+L 4CAN-rescue:.-XZMDKVG55W-8-4CAN-rescue D2
 U 1 1 5F03BD2B
 P 7950 7100
@@
 	6750 7600 7900 7600
 $Comp
-L 4CAN-rescue:.-XZMDKVG55W-8 D3
+L 4CAN-rescue:.-XZMDKVG55W-8-4CAN-rescue D3
 U 1 1 5F1248A2
 P 5300 9750
@@
 $EndComp
 $Comp
-L 4CAN-rescue:.-XZMDKVG55W-8 D4
+L 4CAN-rescue:.-XZMDKVG55W-8-4CAN-rescue D4
 U 1 1 5F1289E0
 P 5300 10950
@@
 	6600 7750 6600 7850
 $Comp
-L 4CAN-rescue:C0805Y103K1RACAUTO-2020-06-11_20-43-35 C2
+L 4CAN-rescue:C0805Y103K1RACAUTO-2020-06-11_20-43-35-4CAN-rescue C2
 U 1 1 5EE38062
 P 5450 7850
@@
 	6150 8550 6800 8550
 $Comp
-L 4CAN-rescue:F930J227MNC-2020-06-11_20-40-41 C1
+L 4CAN-rescue:F930J227MNC-2020-06-11_20-40-41-4CAN-rescue C1
 U 1 1 5EE66B35
 P 5850 7850
@@
 220uf
 $Comp
-L 4CAN-rescue:C0805Y103K1RACAUTO-2020-06-11_20-43-35 C3
+L 4CAN-rescue:C0805Y103K1RACAUTO-2020-06-11_20-43-35-4CAN-rescue C3
 U 1 1 5EEBA3FB
 P 8200 7750
@@
 $EndComp
 $Comp
-L 4CAN-rescue:C0805Y103K1RACAUTO-2020-06-11_20-43-35 C9
+L 4CAN-rescue:C0805Y103K1RACAUTO-2020-06-11_20-43-35-4CAN-rescue C9
 U 1 1 5F1EEF36
 P 6250 14250
@@
 120
 $Comp
-L 4CAN-rescue:ED555_2DS-2020-06-09_21-20-13 J2
+L 4CAN-rescue:ED555_2DS-2020-06-09_21-20-13-4CAN-rescue J2
 U 1 1 5EE39292
 P 17900 3750
@@
 	17700 2350 17900 2350
 $Comp
-L 4CAN-rescue:RC0805FR-07120RL-2020-06-09_18-29-32 R6
+L 4CAN-rescue:RC0805FR-07120RL-2020-06-09_18-29-32-4CAN-rescue R6
 U 1 1 5EE08C55
 P 16300 6150
@@
 $EndComp
 $Comp
-L 4CAN-rescue:RC0805FR-07120RL-2020-06-09_18-29-32 R5
+L 4CAN-rescue:RC0805FR-07120RL-2020-06-09_18-29-32-4CAN-rescue R5
 U 1 1 5EE01523
 P 16200 2950
@@
 $EndComp
 $Comp
-L 4CAN-rescue:ED555_2DS-2020-06-09_21-20-13 J5
+L 4CAN-rescue:ED555_2DS-2020-06-09_21-20-13-4CAN-rescue J5
 U 1 1 5EE3ECFC
 P 17850 13350
@@
 $EndComp
 $Comp
-L 4CAN-rescue:ED555_2DS-2020-06-09_21-20-13 J4
+L 4CAN-rescue:ED555_2DS-2020-06-09_21-20-13-4CAN-rescue J4
 U 1 1 5EE3DB0F
 P 17900 10200
@@
 $EndComp
 $Comp
-L 4CAN-rescue:ED555_2DS-2020-06-09_21-20-13 J3
+L 4CAN-rescue:ED555_2DS-2020-06-09_21-20-13-4CAN-rescue J3
 U 1 1 5EE3C9F4
 P 17900 7000
@@
 $EndComp
 $Comp
-L 4CAN-rescue:RC0805FR-07120RL-2020-06-09_18-29-32 R8
+L 4CAN-rescue:RC0805FR-07120RL-2020-06-09_18-29-32-4CAN-rescue R8
 U 1 1 5EE0A9F7
 P 16500 12500
@@
 $EndComp
 $Comp
-L 4CAN-rescue:RC0805FR-07120RL-2020-06-09_18-29-32 R7
+L 4CAN-rescue:RC0805FR-07120RL-2020-06-09_18-29-32-4CAN-rescue R7
 U 1 1 5EE09C14
 P 16400 9350
@@
 	10350 7900 10200 7900
 $Comp
-L 4CAN-rescue:C0805Y103K1RACAUTO-2020-06-11_20-43-35 C11
+L 4CAN-rescue:C0805Y103K1RACAUTO-2020-06-11_20-43-35-4CAN-rescue C11
 U 1 1 5FBE3D6B
 P 10200 7950
@@
 	10350 4650 10200 4650
 $Comp
-L 4CAN-rescue:C0805Y103K1RACAUTO-2020-06-11_20-43-35 C10
+L 4CAN-rescue:C0805Y103K1RACAUTO-2020-06-11_20-43-35-4CAN-rescue C10
 U 1 1 5FC0B3E6
 P 10200 4700
@@
 	10350 11100 10200 11100
 $Comp
-L 4CAN-rescue:C0805Y103K1RACAUTO-2020-06-11_20-43-35 C12
+L 4CAN-rescue:C0805Y103K1RACAUTO-2020-06-11_20-43-35-4CAN-rescue C12
 U 1 1 5FC24789
 P 10200 11150
@@
 $EndComp
 $Comp
-L 4CAN-rescue:C0805Y103K1RACAUTO-2020-06-11_20-43-35 C13
+L 4CAN-rescue:C0805Y103K1RACAUTO-2020-06-11_20-43-35-4CAN-rescue C13
 U 1 1 5FC40325
 P 10200 14300
@@
 	14750 6800 14600 6800
 $Comp
-L 4CAN-rescue:C0805Y103K1RACAUTO-2020-06-11_20-43-35 C6
+L 4CAN-rescue:C0805Y103K1RACAUTO-2020-06-11_20-43-35-4CAN-rescue C6
 U 1 1 5FC610D5
 P 14600 6850
@@
 	14750 3550 14600 3550
 $Comp
-L 4CAN-rescue:C0805Y103K1RACAUTO-2020-06-11_20-43-35 C5
+L 4CAN-rescue:C0805Y103K1RACAUTO-2020-06-11_20-43-35-4CAN-rescue C5
 U 1 1 5FC7C2EE
 P 14600 3600
@@
 	14750 10000 14600 10000
 $Comp
-L 4CAN-rescue:C0805Y103K1RACAUTO-2020-06-11_20-43-35 C7
+L 4CAN-rescue:C0805Y103K1RACAUTO-2020-06-11_20-43-35-4CAN-rescue C7
 U 1 1 5FC97F31
 P 14600 10050
@@
 	14750 13150 14600 13150
 $Comp
-L 4CAN-rescue:C0805Y103K1RACAUTO-2020-06-11_20-43-35 C8
+L 4CAN-rescue:C0805Y103K1RACAUTO-2020-06-11_20-43-35-4CAN-rescue C8
 U 1 1 5FCB4427
 P 14600 13200
@@
 	12800 3100 14750 3100
 $Comp
-L 4CAN-rescue:RC0805FR-07120RL-2020-06-09_18-29-32 R2
+L 4CAN-rescue:RC0805FR-07120RL-2020-06-09_18-29-32-4CAN-rescue R2
 U 1 1 5F2D685D
 P 9950 6950
@@
 $EndComp
 $Comp
-L 4CAN-rescue:RC0805FR-07120RL-2020-06-09_18-29-32 R1
+L 4CAN-rescue:RC0805FR-07120RL-2020-06-09_18-29-32-4CAN-rescue R1
 U 1 1 5F31E8B1
 P 9950 3700
@@
 $EndComp
 $Comp
-L 4CAN-rescue:RC0805FR-07120RL-2020-06-09_18-29-32 R3
+L 4CAN-rescue:RC0805FR-07120RL-2020-06-09_18-29-32-4CAN-rescue R3
 U 1 1 5F36E072
 P 9950 10150
@@
 $EndComp
 $Comp
-L 4CAN-rescue:RC0805FR-07120RL-2020-06-09_18-29-32 R4
+L 4CAN-rescue:RC0805FR-07120RL-2020-06-09_18-29-32-4CAN-rescue R4
 U 1 1 5F37F26F
 P 9950 13300
